File: hardware/imu81/imu81.kicad_pcb (KiCad board)
At the start: 4 copper layers, 16 x 17 mm, 25 parts, among them J3 Conn_01x06, J4 Conn_01x06, U1 ICM-42670-P, U2 ICM-42670-P, U3 ICM-42670-P, U4 ICM-42670-P, U5 ICM-42670-P, U6 ICM-42670-P, U7 ICM-42670-P, U8 ICM-42670-P, U9 STM32U031K8Ux

Commit message: feat: add workflow
Other:
- board text added: "GND"
- board text added: "INT"
- board text added: "SCL"
- board text added: "SDA"
- board text added: "SWCK"
- board text added: "SWIO"
- board text added: "SWO"
- board text added: "VDD"
- board text added: "imu81 github.com/ arifbalik/imu-array"
- board text added: "nRST"
Changed lines of the file:
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@@
 			(layer "B.Mask"
 				(type "Bottom Solder Mask")
+				(color "Black")
 				(thickness 0.01)
 			)
@@
 			(layer "B.SilkS"
 				(type "Bottom Silk Screen")
+				(color "Yellow")
 			)
 			(copper_finish "HAL lead-free")
@@
 		(layer "Edge.Cuts")
 	)
+	(gr_text "VDD"
+		(at 48.5 77.7 270)
+		(layer "B.SilkS")
+		(effects
+			(font
+				(size 1 1)
+				(thickness 0.2)
+				(bold yes)
+			)
+			(justify left bottom mirror)
+		)
+	)
+	(gr_text "SWCK"
+		(at 48.6 67.2 270)
+		(layer "B.SilkS")
+		(effects
+			(font
+				(size 1 1)
+				(thickness 0.2)
+				(bold yes)
+			)
+			(justify left bottom mirror)
+		)
+	)
+	(gr_text "VDD"
+		(at 40.9 77.7 270)
+		(layer "B.SilkS")
+		(effects
+			(font
+				(size 1 1)
+				(thickness 0.2)
+				(bold yes)
+			)
+			(justify left bottom mirror)
+		)
+	)
+	(gr_text "GND"
+		(at 51.1 77.7 270)
+		(layer "B.SilkS")
+		(effects
+			(font
+				(size 1 1)
+				(thickness 0.2)
+				(bold yes)
+			)
+			(justify left bottom mirror)
+		)
+	)
+	(gr_text "INT"
+		(at 41 65.4 270)
+		(layer "B.SilkS")
+		(effects
+			(font
+				(size 1 1)
+				(thickness 0.2)
+				(bold yes)
+			)
+			(justify left bottom mirror)
+		)
+	)
+	(gr_text "SWO"
+		(at 43.4 66.3 270)
+		(layer "B.SilkS")
+		(effects
+			(font
+				(size 1 1)
+				(thickness 0.2)
+				(bold yes)
+			)
+			(justify left bottom mirror)
+		)
+	)
+	(gr_text "imu81\ngithub.com/\narifbalik/imu-array"
+		(at 53 72.8 0)
+		(layer "B.SilkS")
+		(effects
+			(font
+				(size 1 1)
+				(thickness 0.2)
+				(bold yes)
+			)
+			(justify left bottom mirror)
+		)
+	)
+	(gr_text "SWIO"
+		(at 46.2 66.7 270)
+		(layer "B.SilkS")
+		(effects
+			(font
+				(size 1 1)
+				(thickness 0.2)
+				(bold yes)
+			)
+			(justify left bottom mirror)
+		)
+	)
+	(gr_text "GND"
+		(at 51.3 66.1 270)
+		(layer "B.SilkS")
+		(effects
+			(font
+				(size 1 1)
+				(thickness 0.2)
+				(bold yes)
+			)
+			(justify left bottom mirror)
+		)
+	)
+	(gr_text "nRST"
+		(at 38.4 66.7 270)
+		(layer "B.SilkS")
+		(effects
+			(font
+				(size 1 1)
+				(thickness 0.2)
+				(bold yes)
+			)
+			(justify left bottom mirror)
+		)
+	)
+	(gr_text "SDA"
+		(at 43.4 77.7 270)
+		(layer "B.SilkS")
+		(effects
+			(font
+				(size 1 1)
+				(thickness 0.2)
+				(bold yes)
+			)
+			(justify left bottom mirror)
+		)
+	)
+	(gr_text "SCL"
+		(at 46 77.7 270)
+		(layer "B.SilkS")
+		(effects
+			(font
+				(size 1 1)
+				(thickness 0.2)
+				(bold yes)
+			)
+			(justify left bottom mirror)
+		)
+	)
+	(gr_text "GND"
+		(at 38.4 77.7 270)
+		(layer "B.SilkS")
+		(effects
+			(font
+				(size 1 1)
+				(thickness 0.2)
+				(bold yes)
+			)
+			(justify left bottom mirror)
+		)
+	)
 	(gr_text "No"
 		(at 154.357138 74.171 0)
@@
 	)
 	(segment
-		(start 41.100011 67.999995)
-		(end 41.100001 67)
-		(width 0.1)
-		(layer "B.Cu")
-		(net 6)
-	)
-	(segment
 		(start 49.8 74.1)
 		(end 49.8 72.800001)
@@
 	)
 	(segment
-		(start 41.600008 68.900008)
-		(end 41.600008 68.499992)
-		(width 0.1)
-		(layer "B.Cu")
-		(net 6)
-	)
-	(segment
-		(start 41.100001 67)
-		(end 41.499993 66.599983)
-		(width 0.1)
-		(layer "B.Cu")
-		(net 6)
-	)
-	(segment
 		(start 42.1 66.6)
 		(end 42.999999 66.6)
@@
 	)
 	(segment
-		(start 41.600008 68.499992)
-		(end 41.100011 67.999995)
+		(start 49.4 71.8)
+		(end 49.399987 72.400005)
 		(width 0.1)
 		(layer "B.Cu")
@@
 	)
 	(segment
-		(start 49.4 71.8)
-		(end 49.399987 72.400005)
+		(start 41.65 68.95)
+		(end 41.600008 68.900008)
 		(width 0.1)
 		(layer "B.Cu")
@@
 	)
 	(segment
-		(start 41.65 68.95)
-		(end 41.600008 68.900008)
+		(start 49.800001 70.7)
+		(end 50.100013 70.400005)
 		(width 0.1)
 		(layer "B.Cu")
@@
 	)
 	(segment
-		(start 49.800001 70.7)
-		(end 50.100013 70.400005)
+		(start 45.1 73.1)
+		(end 44.7 73.5)
 		(width 0.1)
 		(layer "B.Cu")
@@
 	)
 	(segment
-		(start 45.1 73.1)
-		(end 44.7 73.5)
+		(start 41.100011 67.999995)
+		(end 41.100011 66.899983)
+		(width 0.1)
+		(layer "B.Cu")
+		(net 6)
+	)
+	(segment
+		(start 41.600008 68.499992)
+		(end 41.100011 67.999995)
 		(width 0.1)
 		(layer "B.Cu")
@@
 	)
 	(segment
+		(start 41.399994 66.6)
+		(end 42.1 66.6)
+		(width 0.1)
+		(layer "B.Cu")
+		(net 6)
+	)
+	(segment
 		(start 42.999999 66.6)
 		(end 43.199997 66.399992)
@@
 	)
 	(segment
+		(start 41.100011 66.899983)
+		(end 41.399994 66.6)
+		(width 0.1)
+		(layer "B.Cu")
+		(net 6)
+	)
+	(segment
 		(start 48.8 74.3)
 		(end 49.6 74.3)
@@
 	)
 	(segment
-		(start 41.499993 66.599983)
-		(end 42.1 66.6)
-		(width 0.1)
-		(layer "B.Cu")
-		(net 6)
-	)
-	(segment
 		(start 45.85 66.449999)
 		(end 47.05 66.45)
@@
 	)
 	(segment
+		(start 41.600008 68.900008)
+		(end 41.600008 68.499992)
+		(width 0.1)
+		(layer "B.Cu")
+		(net 6)
+	)
+	(segment
 		(start 49.399987 72.400005)
 		(end 49.699999 72.7)
@@
 	)
 	(segment
+		(start 40.5 67)
+		(end 41.7 65.8)
+		(width 0.1)
+		(layer "B.Cu")
+		(net 10)
+	)
+	(segment
+		(start 40.5 69.6)
+		(end 40.5 67)
+		(width 0.1)
+		(layer "B.Cu")
+		(net 10)
+	)
+	(segment
 		(start 41.8 65.399999)
 		(end 41.749994 65.350014)
@@
 	)
 	(segment
-		(start 41.7 65.35)
-		(end 41.7 65.999999)
-		(width 0.1)
-		(layer "B.Cu")
-		(net 10)
-	)
-	(segment
 		(start 48.2 75.5)
 		(end 49.4 75.5)
@@
 	)
 	(segment
-		(start 49.599999 66.600001)
-		(end 48.400004 65.399989)
+		(start 41.7 65.8)
+		(end 41.7 65.35)
 		(width 0.1)
 		(layer "B.Cu")
@@
 	)
 	(segment
-		(start 40.80001 71.4)
-		(end 40.80001 73.90001)
+		(start 49.599999 66.600001)
+		(end 48.400004 65.399989)
 		(width 0.1)
 		(layer "B.Cu")
@@
 	)
 	(segment
-		(start 40.499999 67.2)
-		(end 41.7 65.999999)
+		(start 40.80001 71.4)
+		(end 40.80001 73.90001)
 		(width 0.1)
 		(layer "B.Cu")
@@
 		(width 0.1)
 		(layer "B.Cu")
-		(net 10)
-	)
-	(segment
-		(start 40.499999 67.2)
-		(end 40.5 69.6)
-		(width 0.1)
-		(layer "B.Cu")
